File: keyboard.kicad_pcb (KiCad board)
At the start: 2 copper layers, 130.6 x 150.1 mm, 170 parts, among them P1 USB_B, P10 CONN_01X01, P11 CONN_01X01, P12 CONN_01X01, P13 CONN_01X01, P2 CONN_02X03, P3 CONN_01X01, P4 CONN_01X01, P5 CONN_01X01, P6 CONN_01X01, P7 CONN_01X01, P8 CONN_01X01, P9 CONN_01X01, SW10 SW_PUSH, SW11 SW_PUSH, SW12 SW_PUSH, SW13 SW_PUSH, SW14 SW_PUSH, SW15 SW_PUSH, SW2 SW_PUSH, SW24 SW_PUSH, SW25 SW_PUSH, SW26 SW_PUSH, SW27 SW_PUSH, SW28 SW_PUSH, SW29 SW_PUSH, SW3 SW_PUSH, SW30 SW_PUSH, SW31 SW_PUSH, SW32 SW_PUSH, SW33 SW_PUSH, SW34 SW_PUSH, SW35 SW_PUSH, SW36 SW_PUSH, SW37 SW_PUSH, SW4 SW_PUSH, SW5 SW_PUSH, SW6 SW_PUSH, SW7 SW_PUSH, SW8 SW_PUSH, SW9 SW_PUSH, U1 ATmega32U4, X1 CRYSTAL_SMD

Commit message: sent to fab
Other:
- board text added: "shortcut prototype v0.4 12/16"
- board text removed: "shortcut prototype v0.1"
Changed lines of the file:
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@@
       (net 1 Earth) (zone_connect 2))
+  )
+  (gr_text "shortcut prototype v0.4 12/16" (at 77.5 27 180) (layer F.SilkS)
+    (effects (font (size 1.5 1.5) (thickness 0.3)))
   )
   (gr_text "0v\nc6\n+5\nr4\nljy\nr3\nljx\nr2\nc7\nr1" (at 58.5 33 180) (layer F.SilkS)
@@
     (effects (font (size 1.5 1.5) (thickness 0.3)) (justify mirror))
   )
-  (gr_text "shortcut prototype v0.1" (at 86 27.5 180) (layer F.SilkS)
+  (gr_text "shortcut prototype v0.4 12/16" (at 86 172.5) (layer F.SilkS)
     (effects (font (size 1.5 1.5) (thickness 0.3)))
   )
-  (gr_text "shortcut prototype v0.1" (at 81 172.5) (layer F.SilkS)
-    (effects (font (size 1.5 1.5) (thickness 0.3)))
-  )

Commit message: v5 switches routed + outline
Parts:
- removed ? (x44): via, fp:via
- removed C4: 1u, Capacitors_SMD:C_0805
- removed D37 (x2), D38 (x2), D39 (x2), D40 (x2), D41 (x2), D42 (x2), D43 (x2), D44 (x2): D, Diodes_SMD:SOD-123
- removed P13 (x2): CONN_01X01, Mounting_Holes:MountingHole_4mm
- removed S3 (x2), S4 (x2): alps_4way, fp:alps 4way smt
- removed thumb-l2 (x2), thumb1, thumb2: CONN_02X05, fp:thumbpad connector
- added D45: D, Diodes_SMD:SOD-123, F.Cu at (137.2, 164.1)
- added D46: D, Diodes_SMD:SOD-123, F.Cu at (144.3, 83.0)
- added P15: CONN_01X06, Pin_Headers:Pin_Header_Straight_1x06, F.Cu at (37.0, 145.2)
- added P18: CONN_01X06, Pin_Headers:Pin_Header_Straight_1x06, F.Cu at (264.0, 70.2)
- added P6: CONN_01X01, Mounting_Holes:MountingHole_4mm, F.Cu at (27.9, 97.0)
- added SW1: SW_PUSH, fp:CHERRY_MXx4, F.Cu at (147.0, 153.0)
- added SW16: SW_PUSH, fp:CHERRY_MXx4, F.Cu at (153.9, 78.0)
- P1: value USB_B -> USB_OTG
- SW10, SW2, SW24, SW25, SW26, SW27, SW28, SW29, SW3, SW30, SW31, SW32, SW4, SW5, SW6, SW7, SW8, SW9: footprint fp:CHERRY_MX -> fp:CHERRY_MXx4
- SW11, SW12, SW13, SW14, SW15, SW33, SW34, SW35, SW36, SW37: footprint fp:CHERRY_MX -> fp:CHERRY_MXx2
- moved P8 233.4 mm to (272.0, 68.7)
- moved conn2 213.3 mm to (245.8, 28.0), turned to 0 degrees
- moved SW36 208.8 mm to (258.6, 38.1), turned to 357.5 degrees
- moved SW37 204.2 mm to (257.7, 57.7), turned to 357.5 degrees
- moved D36 197.8 mm to (247.5, 54.0), turned to 270 degrees
- moved D35 196.1 mm to (248.9, 33.3), turned to 270 degrees
- moved SW33 171.4 mm to (238.6, 36.4), turned to 357.5 degrees
- moved led9 168.6 mm to (248.3, 42.5), turned to 180 degrees
- moved SW35 167.9 mm to (236.9, 75.6), turned to 357.5 degrees
- moved SW34 165.3 mm to (237.8, 56.0), turned to 357.5 degrees
- moved P9 157.3 mm to (273.0, 22.0)
- moved D34 155.4 mm to (228.6, 75.9), turned to 270 degrees
- moved D32 153.3 mm to (230.0, 33.9), turned to 270 degrees
- moved D33 146.5 mm to (229.2, 54.3)
- moved led11 145.1 mm to (227.3, 67.0), turned to 180 degrees
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Connections:
- P1 pad 4: Earth -> (no net)
- P1 pad 5: (no net) -> Earth
- P1 pad 6: (no net) -> Net-(P1-Pad6)
- U1 pad 38: /r-joy-y -> (no net)
- U1 pad 39: /r-joy-x -> (no net)
- U1 pad 40: /l-joy-y -> (no net)
- U1 pad 41: /l-joy-x -> (no net)
- U1 pad 42: Net-(C4-Pad1) -> (no net)
- conn1 pad 12: /l-joy-x -> (no net)
- conn1 pad 14: /l-joy-y -> (no net)
- conn2 pad 3: /l-l-joy-y -> (no net)
- conn2 pad 5: /l-l-joy-x -> (no net)
- led1 pad 4: Net-(led1-Pad4) -> /ws2812
- led10 pad 2: (no net) -> Net-(led10-Pad2)
- led11 pad 4: Net-(led11-Pad4) -> Net-(led10-Pad2)
- led12 pad 2: Net-(led10-Pad4) -> Net-(led12-Pad2)
- led12 pad 4: Net-(led12-Pad4) -> Net-(led11-Pad2)
- led13 pad 2: Net-(led11-Pad4) -> Net-(led13-Pad2)
- led13 pad 4: Net-(led13-Pad4) -> Net-(led12-Pad2)
- led14 pad 2: Net-(led12-Pad4) -> Net-(led14-Pad2)
- led14 pad 4: Net-(led14-Pad4) -> Net-(led13-Pad2)
- led15 pad 2: Net-(led13-Pad4) -> Net-(led15-Pad2)
- led15 pad 4: /l-ws2812-out -> Net-(led14-Pad2)
- led16 pad 2: Net-(led14-Pad4) -> (no net)
- led16 pad 4: Net-(led16-Pad4) -> Net-(led15-Pad2)
- led2 pad 2: /ws2812-out -> Net-(led2-Pad2)
- led2 pad 4: Net-(led2-Pad4) -> Net-(led1-Pad2)
- led3 pad 2: Net-(led1-Pad4) -> Net-(led3-Pad2)
- led3 pad 4: Net-(led3-Pad4) -> Net-(led2-Pad2)
- led4 pad 2: Net-(led2-Pad4) -> Net-(led4-Pad2)
- led4 pad 4: Net-(led4-Pad4) -> Net-(led3-Pad2)
- led5 pad 2: Net-(led3-Pad4) -> Net-(led5-Pad2)
- led5 pad 4: Net-(led5-Pad4) -> Net-(led4-Pad2)
- led6 pad 2: Net-(led4-Pad4) -> Net-(led6-Pad2)
- led6 pad 4: Net-(led6-Pad4) -> Net-(led5-Pad2)
- led7 pad 2: Net-(led5-Pad4) -> Net-(led7-Pad2)
- led7 pad 4: /ws2812 -> Net-(led6-Pad2)
- led8 pad 2: Net-(led6-Pad4) -> /ws2812-out
- led8 pad 4: Net-(led1-Pad2) -> Net-(led7-Pad2)
- led9 pad 2: Net-(led16-Pad4) -> Net-(led10-Pad4)
- led9 pad 4: Net-(led11-Pad2) -> /l-ws2812-out
Routing:
- net Earth: track 347.5 -> 173.9 mm, vias 34 -> 12
- net /r-joy-x: track 149.8 -> 0.00 mm, vias 2 -> 0
- net /l-col5: track 34.0 -> 173.2 mm
- net /r-joy-y: track 130.1 -> 0.00 mm, vias 4 -> 0
- net /l-joy-y: track 120.7 -> 0.00 mm, vias 2 -> 0
- net /col12: track 125.9 -> 235.5 mm
- net /l-joy-x: track 108.0 -> 0.00 mm, vias 2 -> 0
- net /left keys/thumb/row1: track 75.7 -> 0.00 mm, vias 4 -> 0
- net /col13: track 108.7 -> 184.4 mm, vias 2 -> 1
- net /l-row3: track 163.1 -> 236.2 mm, vias 8 -> 6
- net /left keys/thumb/col2: track 67.3 -> 0.00 mm
- net /col14: track 125.7 -> 185.6 mm
- net /left keys/thumb/col1: track 52.9 -> 0.00 mm
- net /l-l-joy-y: track 51.2 -> 0.00 mm, vias 1 -> 0
- net Net-(led3-Pad4): track 50.9 -> 0.00 mm, vias 6 -> 0
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Other:
- board outline removed
- board text added: "89"
- board text added: "shortcut prototype v0.5 1/17"
- board text removed: "0v c6 +5 r4 ljy r3 ljx r2 c7 r1"
- board text removed: "left side"
- board text removed: "r1 c14 r2 ljx r3 rjy r4 +5 c13 0v"
- board text removed: "shortcut prototype thumboard v0.1"
- board text removed: "shortcut prototype v0.4 12/16"

Commit message: v5 prefab
Parts:
- added D15: D, Diodes_SMD:SOD-123, F.Cu at (260.6, 139.5)
- added D15: D, Diodes_SMD:SOD-123, F.Cu at (218.8, 140.0)
- added D16: D, Diodes_SMD:SOD-123, F.Cu at (262.8, 139.5)
- added D16: D, Diodes_SMD:SOD-123, F.Cu at (221.0, 140.0)
- added D17: D, Diodes_SMD:SOD-123, F.Cu at (242.5, 139.5)
- added D17: D, Diodes_SMD:SOD-123, F.Cu at (200.8, 140.0)
- added D18: D, Diodes_SMD:SOD-123, F.Cu at (244.6, 139.5)
- added D18: D, Diodes_SMD:SOD-123, F.Cu at (202.8, 140.0)
- added D19: D, Diodes_SMD:SOD-123, F.Cu at (242.5, 123.5)
- added D19: D, Diodes_SMD:SOD-123, F.Cu at (200.8, 124.0)
- added D20: D, Diodes_SMD:SOD-123, F.Cu at (262.8, 123.5)
- added D20: D, Diodes_SMD:SOD-123, F.Cu at (221.0, 124.0)
- added D21: D, Diodes_SMD:SOD-123, F.Cu at (260.6, 123.5)
- added D21: D, Diodes_SMD:SOD-123, F.Cu at (218.8, 124.0)
- added D22: D, Diodes_SMD:SOD-123, F.Cu at (244.6, 123.5)
- added D22: D, Diodes_SMD:SOD-123, F.Cu at (202.8, 124.0)
- added P13: CONN_01X01, Mounting_Holes:MountingHole_4mm, F.Cu at (260.6, 131.5)
- added P13: CONN_01X01, Mounting_Holes:MountingHole_4mm, F.Cu at (218.8, 132.0)
- added P16: CONN_01X06, Pin_Headers:Pin_Header_Straight_1x06, F.Cu at (258.7, 145.5)
- added P16: CONN_01X06, Pin_Headers:Pin_Header_Straight_1x06, F.Cu at (216.9, 146.0)
- added P17: CONN_01X01, Mounting_Holes:MountingHole_4mm, F.Cu at (244.6, 131.5)
- added P17: CONN_01X01, Mounting_Holes:MountingHole_4mm, F.Cu at (202.8, 132.0)
- added P3: CONN_01X01, Mounting_Holes:MountingHole_4mm, F.Cu at (194.8, 23.3)
- added REF**: via, fp:via, F.Cu at (184.2, 55.0)
- added REF**: via, fp:via, F.Cu at (237.0, 49.8)
- added REF**: via, fp:via, F.Cu at (141.8, 69.2)
- added REF**: via, fp:via, F.Cu at (116.2, 138.2)
- added REF**: via, fp:via, F.Cu at (83.2, 166.0)
- added REF**: via, fp:via, F.Cu at (149.2, 49.8)
- added REF**: via, fp:via, F.Cu at (237.0, 44.8)
- added REF**: via, fp:via, F.Cu at (227.5, 60.2)
- added REF**: via, fp:via, F.Cu at (111.2, 100.2)
- added REF**: via, fp:via, F.Cu at (155.2, 123.0)
- added REF**: via, fp:via, F.Cu at (174.2, 37.5)
- added REF**: via, fp:via, F.Cu at (208.8, 90.8)
- added REF**: via, fp:via, F.Cu at (229.0, 90.8)
- added REF**: via, fp:via, F.Cu at (31.0, 137.8)
- added REF**: via, fp:via, F.Cu at (62.0, 124.8)
- added REF**: via, fp:via, F.Cu at (203.8, 90.8)
- added REF**: via, fp:via, F.Cu at (71.0, 111.8)
- added REF**: via, fp:via, F.Cu at (184.2, 50.0)
- added REF**: via, fp:via, F.Cu at (141.8, 74.2)
- added REF**: via, fp:via, F.Cu at (95.8, 111.8)
- added REF**: via, fp:via, F.Cu at (41.2, 123.2)
- added REF**: via, fp:via, F.Cu at (154.2, 49.8)
- added S1: alps_4way, fp:alps 4way smt, F.Cu at (252.6, 139.0)
- added S1: alps_4way, fp:alps 4way smt, F.Cu at (210.8, 139.5)
- added S2: alps_4way, fp:alps 4way smt, F.Cu at (252.6, 124.0)
- added S2: alps_4way, fp:alps 4way smt, F.Cu at (210.8, 124.5)
- moved P15 12.6 mm to (49.7, 145.2), turned to 270 degrees
Routing:
- net /right keys/thumb/row3: track 0.00 -> 73.7 mm, vias 0 -> 2
- net /right keys/thumb/row1: track 0.00 -> 71.6 mm, vias 0 -> 4
- net /right keys/thumb/row2: track 0.00 -> 63.5 mm, vias 0 -> 4
- net /right keys/thumb/row4: track 0.00 -> 61.8 mm, vias 0 -> 4
- net /right keys/thumb/col2: track 0.00 -> 54.6 mm, vias 0 -> 2
- net Earth: track 173.9 -> 226.3 mm, vias 12 -> 15
- net Net-(D19-Pad2): track 0.00 -> 38.6 mm
- net Net-(D17-Pad2): track 0.00 -> 32.2 mm
- net /right keys/thumb/col1: track 0.00 -> 25.7 mm, vias 0 -> 2
- net Net-(D15-Pad2): track 0.00 -> 18.5 mm
- net /col14: track 185.6 -> 202.6 mm, vias 3 -> 5
- net Net-(P1-Pad6): track 0.00 -> 13.5 mm
- net Net-(D20-Pad2): track 0.00 -> 13.2 mm
- net Net-(D16-Pad2): track 0.00 -> 13.2 mm
- net /col13: track 184.4 -> 195.8 mm
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Other:
- board outline added: 434.7 x 179.9 mm
- board text removed: "89"

Commit message: sent to fab
Parts:
- moved D15 176.5 mm to (46.1, 176.0)
- moved D16 176.5 mm to (48.2, 176.0)
- moved D17 176.5 mm to (28.0, 176.0)
- moved D18 176.5 mm to (30.1, 176.0)
- moved D19 176.5 mm to (28.0, 160.0)
- moved D20 176.5 mm to (48.2, 160.0)
- moved D21 176.5 mm to (46.1, 160.0)
- moved D22 176.5 mm to (30.1, 160.0)
- moved P13 176.5 mm to (46.0, 168.0)
- moved P16 176.5 mm to (44.2, 182.0)
- moved P17 176.5 mm to (30.1, 168.0)
- moved S1 176.5 mm to (38.1, 175.5)
- moved S2 176.5 mm to (38.1, 160.5)
- moved D15 113.8 mm to (158.6, 89.0)
- moved D16 113.8 mm to (160.8, 89.0)
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Other:
- board size 434.7 x 179.9 mm -> 323.7 x 193.9 mm
